File: KiCAD Files/BoardGame/Battery charger.kicad_sch (KiCad schematic)
At the start: 15 parts, among them J301 Conn_01x01, J302 Conn_01x01, U301 MCP73871-2CC

Commit message: update
Connections:
- net PG: no longer names the net of U301.6 (~{PG})
- net STAT1: no longer names the net of U301.8 (STAT1/~{LBO})
- net STAT2: no longer names the net of U301.7 (STAT2)
- no-connect marks 0 -> 3
Other:
- moved on the sheet: C301, C302, C303, C304, R301, R302, R303, R307, R308, R310, U301
