File: KiCAD Files/BoardGame/Touchpad LEDs.kicad_sch (KiCad schematic)
At the start: 13 parts

Commit message: update
Other:
- moved on the sheet: D1085, D1086, D1087, D1088, D1089, D1090, D1091, D1092, D1093, D1094, D1095, D1096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

Commit message: update
Other:
- moved on the sheet: D1085, D1086, D1087, D1088, D1089, D1090, D1091, D1092, D1093, D1094, D1095, D1096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
