File: KiCAD Files/BoardGame/Mechanical.kicad_sch (KiCad schematic)
At the start: 8 parts

Commit message: update
Parts:
- removed H1005, H1006, H1007, H1008: MountingHole, MountingHole:MountingHole_3.2mm_M3, symbol Mechanical:MountingHole
