File: KiCAD Files/BoardGame/Displays.kicad_sch (KiCad schematic)
At the start: 5 parts

Commit message: update
Parts:
- U1091: footprint (none) -> Footprints:GC9A01
Changed lines of the file:
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@@
 			)
 		)
-		(property "Footprint" ""
+		(property "Footprint" "Footprints:GC9A01"
 			(at 190.5 114.3 0)
 			(effects

Commit message: update
Parts:
- U1087, U1088, U1089, U1090: footprint (none) -> Footprints:OLED 1.3inch
Changed lines of the file:
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@@
 			)
 		)
-		(property "Footprint" ""
+		(property "Footprint" "Footprints:OLED 1.3inch"
 			(at 138.43 111.76 0)
 			(effects
@@
 			)
 		)
-		(property "Footprint" ""
+		(property "Footprint" "Footprints:OLED 1.3inch"
 			(at 123.19 111.76 0)
 			(effects
@@
 			)
 		)
-		(property "Footprint" ""
+		(property "Footprint" "Footprints:OLED 1.3inch"
 			(at 153.67 111.76 0)
 			(effects
@@
 			)
 		)
-		(property "Footprint" ""
+		(property "Footprint" "Footprints:OLED 1.3inch"
 			(at 168.91 111.76 0)
 			(effects

Commit message: update
Parts:
- U1087, U1088, U1089, U1090: footprint Footprints:OLED 1.3inch -> Footprints:OLED 0.96inch
Changed lines of the file:
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@@
 			)
 		)
-		(property "Footprint" "Footprints:OLED 1.3inch"
+		(property "Footprint" "Footprints:OLED 0.96inch"
 			(at 138.43 111.76 0)
 			(effects
@@
 			)
 		)
-		(property "Footprint" "Footprints:OLED 1.3inch"
+		(property "Footprint" "Footprints:OLED 0.96inch"
 			(at 123.19 111.76 0)
 			(effects
@@
 			)
 		)
-		(property "Footprint" "Footprints:OLED 1.3inch"
+		(property "Footprint" "Footprints:OLED 0.96inch"
 			(at 153.67 111.76 0)
 			(effects
@@
 			)
 		)
-		(property "Footprint" "Footprints:OLED 1.3inch"
+		(property "Footprint" "Footprints:OLED 0.96inch"
 			(at 168.91 111.76 0)
 			(effects
