File: KiCAD Files/BoardGame/Path LEDs.kicad_sch (KiCad schematic)
At the start: 53 parts

Commit message: update
Other:
- moved on the sheet: D1011, D1012, D1013, D1014, D1015, D1016, D1017, D1018, D1019, D1020, D1021, D1022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

Commit message: update
Parts:
- removed D1049, D1050, D1051, D1052: WS2812B, Footprints:LED_WS2812B_edited, symbol LED:WS2812B
