File: KiCAD Files/BoardGame/BoardGame.kicad_pcb (KiCad board)
At the start: 2 copper layers, 150 x 150 mm, 218 parts, among them J201 USB_C_Receptacle_USB2.0, J301 Conn_01x01, J302 Conn_01x01, J401 Conn_02x03_Odd_Even, J402 Conn_02x03_Odd_Even, J403 Conn_02x03_Odd_Even, J404 Conn_02x03_Odd_Even, J405 Conn_01x02_Female, J406 Conn_01x02_Female, J407 Conn_01x02_Female, J408 Conn_01x02_Female, J501 USBasp, SW501 SW_Push, U201 USBLC6-2SC6, U202 CH340C, U301 MCP73871-2CC, U401 PCF8575, U501 ATmega328P-A, U601 MT3608, Y501 16MHz

Commit message: update
Parts:
- removed C1001, C1002, C1003, C1004, C1005, C1006, C1007, C1008, C1009: 100n, Capacitor_SMD:C_0603_1608Metric
- removed D1053, D1054, D1055, D1056, D1057, D1058, D1059, D1060, D1061, D1062, D1063, D1064, D1065, D1066, D1067, D1068, D1069, D1070, D1071, D1072, D1073, D1074, D1075, D1076, D1077, D1078, D1079, D1080, D1081, D1082, D1083, D1084: WS2812B, Footprints:LED_WS2812B_edited
- removed D1097, D1098, D1099, D1100, D1101, D1102, D1103, D1104, D1105, D1106: WS2812B, Footprints:WS2812-mini
- removed R1001, R1003, R1004, R1006: 470R, Resistor_SMD:R_0603_1608Metric
Connections:
- U501 pad 10: /Microcontroller/NP_4 -> unconnected-(U501-PD6-Pad10)
- U501 pad 12: /Finish LEDs/NP_1 -> unconnected-(U501-PB0-Pad12)
- U501 pad 26: /Battery indicator LED/NP_6 -> unconnected-(U501-PC3-Pad26)
- U501 pad 9: /Dice LEDs/NP_3 -> unconnected-(U501-PD5-Pad9)
Routing:
- net (no net): track 17.0 -> 1103.0 mm, vias 0 -> 42
- net Net-(D1056-DOUT): track 124.6 -> 0.00 mm, vias 6 -> 0
- net Net-(D1064-DOUT): track 120.2 -> 0.00 mm, vias 4 -> 0
- net Net-(D1080-DOUT): track 100.5 -> 0.00 mm, vias 8 -> 0
- net Net-(D1076-DOUT): track 87.0 -> 0.00 mm, vias 4 -> 0
- net Net-(D1060-DOUT): track 86.3 -> 0.00 mm, vias 4 -> 0
- net Net-(D1072-DOUT): track 84.6 -> 0.00 mm, vias 4 -> 0
- net Net-(D1053-DIN): track 78.6 -> 0.00 mm, vias 3 -> 0
- net Net-(D1069-DIN): track 66.4 -> 0.00 mm, vias 5 -> 0
- net Net-(D1097-DIN): track 56.9 -> 0.00 mm, vias 1 -> 0
- net Net-(D1106-DIN): track 42.0 -> 0.00 mm, vias 3 -> 0
- net unconnected-(U501-PB0-Pad12): track 0.00 -> 20.3 mm, vias 0 -> 2
- net /Finish LEDs/NP_1: track 20.3 -> 0.00 mm, vias 2 -> 0
- net Net-(D1057-DOUT): track 15.5 -> 0.00 mm
- net Net-(D1065-DOUT): track 15.2 -> 0.00 mm
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
Commit message: update
Parts:
- removed C204: 100n, Capacitor_SMD:C_0603_1608Metric
- removed C601, C602: 22u / 16V, Capacitor_SMD:C_1210_3225Metric
- removed D501, D601: SS12, Diode_SMD:D_SMA
- removed J405, J406, J407, J408: Conn_01x02_Female, Connector_PinHeader_1.27mm:PinHeader_1x02_P1.27mm_Vertical
- removed J501: USBasp, Connector_PinHeader_1.27mm:PinHeader_2x03_P1.27mm_Vertical_SMD
- removed L601: 4R7, Footprints:Inductor_4mm(5x5mm pads)
- removed R601: 100k, Resistor_SMD:R_0603_1608Metric
- removed R602: 13k3, Resistor_SMD:R_0603_1608Metric
- removed U501: ATmega328P-A, Package_QFP:TQFP-32_7x7mm_P0.8mm
- removed U601: MT3608, Package_TO_SOT_SMD:SOT-23-6
- removed Y501: 16MHz, Footprints:CSTCE16M0V53-R0
- removed kibuzzard-635CF483: G***, kibuzzard-635CF483
- removed kibuzzard-635CF4BC: G***, kibuzzard-635CF4BC
- removed kibuzzard-635CF4CF: G***, kibuzzard-635CF4CF
- removed kibuzzard-635CF4E4: G***, kibuzzard-635CF4E4
- removed kibuzzard-635CF507: G***, kibuzzard-635CF507
- removed kibuzzard-636375F6: G***, kibuzzard-636375F6
- added C1085: 1uF / 50V, Capacitor_SMD:C_0805_2012Metric, F.Cu at (257.6, 107.5)
- added C1086: 1uF / 50V, Capacitor_SMD:C_0805_2012Metric, F.Cu at (257.6, 110.5)
- added Q1085: UMH3N, Package_TO_SOT_SMD:SOT-363_SC-70-6, B.Cu at (245.7, 108.6)
- added U1085: ESP32-WROOM-32D, Footprints:ESP32, B.Cu at (133.1, 145.9)
- added U1086: XC6210B332MR, Package_TO_SOT_SMD:SOT-23-5, B.Cu at (252.4, 108.2)
- moved R401 148.4 mm to (247.7, 82.0)
- moved R402 148.4 mm to (243.7, 82.0)
- moved C401 148.4 mm to (242.9, 75.8)
- moved U401 140.9 mm to (246.0, 92.3)
- moved C501 114.8 mm to (250.4, 70.2)
- moved C502 114.8 mm to (251.2, 63.2)
- moved R1002 114.8 mm to (261.7, 76.0)
- moved R1005 114.8 mm to (246.9, 68.0)
- moved R501 114.8 mm to (236.7, 73.0)
- moved SW501 114.8 mm to (236.4, 68.7)
- moved LS501 52.7 mm to (261.0, 92.0)
- moved C201 16.2 mm to (117.2, 137.2)
- moved C202 16.2 mm to (110.0, 130.5)
- moved C203 16.2 mm to (110.0, 127.8)
- moved U202 16.2 mm to (110.0, 136.9)
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Connections:
- net /IO Expander/SCL renamed /Displays/SCL0
- net /IO Expander/SDA renamed /Displays/SDA0
- net /USB/USB renamed /USB-UART/USB
- C201 pad 1: Net-(U202-V3) -> Net-(U202-VCC)
- C401 pad 1: +5V -> +3V3
- C501 pad 1: Net-(D501-K) -> +3V3
- C502 pad 1: Net-(D501-K) -> +3V3
- J401 pad 3: +5V -> +3V3
- J401 pad 4: +5V -> +3V3
- J402 pad 3: +5V -> +3V3
- J402 pad 4: +5V -> +3V3
- J403 pad 3: +5V -> +3V3
- J403 pad 4: +5V -> +3V3
- J404 pad 3: +5V -> +3V3
- J404 pad 4: +5V -> +3V3
- LS501 pad 1: Net-(U501-PB2) -> /Microcontroller/IO13
- R401 pad 1: +5V -> +3V3
- R402 pad 1: +5V -> +3V3
- R501 pad 2: +5V -> +3V3
- U202 pad 13: Net-(U202-~{DTR}) -> DTR
- U202 pad 14: unconnected-(U202-~{RTS}-Pad14) -> RTS
- U202 pad 16: VBUS -> Net-(U202-VCC)
- U202 pad 4: Net-(U202-V3) -> VBUS
- U301 pad 6: /Battery charger/PG -> unconnected-(U301-~{PG}-Pad6)
- U301 pad 7: /Battery charger/STAT2 -> unconnected-(U301-STAT2-Pad7)
- U301 pad 8: /Battery charger/STAT1 -> unconnected-(U301-STAT1/~{LBO}-Pad8)
- U401 pad 17: TP_13 -> unconnected-(U401-P14-Pad17)
- U401 pad 24: +5V -> +3V3
Routing:
- net VCC: track 1599.0 -> 0.00 mm, vias 11 -> 0
- net (no net): track 1103.0 -> 0.00 mm, vias 42 -> 0
- net +5V: track 644.5 -> 0.00 mm, vias 16 -> 0
- net VBUS: track 193.6 -> 8.15 mm, vias 4 -> 2
- net TP_11: track 157.3 -> 0.00 mm, vias 2 -> 0
- net TP_12: track 152.1 -> 0.00 mm
- net TP_8: track 138.9 -> 0.00 mm
- net TP_7: track 138.5 -> 0.00 mm
- net TP_9: track 130.0 -> 0.00 mm, vias 2 -> 0
- net /Microcontroller/RESET: track 114.9 -> 0.00 mm, vias 8 -> 0
- net Net-(D1085-DIN): track 108.1 -> 0.00 mm, vias 3 -> 0
- net TP_6: track 98.7 -> 0.00 mm
- net TP_5: track 95.5 -> 0.00 mm
- net Net-(D1093-DOUT): track 93.1 -> 0.00 mm, vias 2 -> 0
- net TP_10: track 92.7 -> 0.00 mm, vias 8 -> 0
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- removed copper zone on B.Cu, net +5V
- removed copper zone on B.Cu, net /Boost Converter/L_OUT
- removed copper zone on B.Cu, net VCC

Commit message: update
Parts:
- added U1091: ~, Footprints:GC9A01, F.Cu at (144.5, 90.3)

Commit message: update
Parts:
- removed H1005, H1006, H1007, H1008: MountingHole, MountingHole:MountingHole_3.2mm_M3
- moved U1091 3.34 mm to (144.0, 87.0)

Commit message: update
Parts:
- added U1087: ~, Footprints:OLED 0.96inch, F.Cu at (144.0, 127.0)
- added U1088: ~, Footprints:OLED 0.96inch, F.Cu at (46.3, 68.7)
- added U1089: ~, Footprints:OLED 0.96inch, F.Cu at (46.3, 103.2)
- added U1090: ~, Footprints:OLED 0.96inch, F.Cu at (46.3, 137.8)
- moved D1039 15.0 mm to (164.6, 116.2)
- moved D1041 15.0 mm to (123.3, 116.4)
- moved D1052 15.0 mm to (114.8, 107.6)
- moved D1038 10.0 mm to (167.2, 128.0)
- moved D1042 10.0 mm to (120.7, 128.1)
- moved D1051 10.0 mm to (103.0, 110.2)
- moved D1037 5.00 mm to (171.7, 139.0)
- moved D1043 5.00 mm to (116.2, 139.0)
- moved D1050 5.00 mm to (91.9, 114.7)

Commit message: update
Parts:
- removed the D1001 at (125.4, 87.0)
- removed the D1014 at (144.0, 68.4)
- removed the D1027 at (162.6, 87.0)
- removed the D1040 at (144.0, 105.6)
- C1085, C1086: moved to B.Cu
- moved U1090 149.7 mm to (187.1, 87.0), turned to 90 degrees
- moved Q1085 147.5 mm to (100.5, 134.5), turned to -90 degrees
- moved U1089 114.3 mm to (144.0, 43.9), turned to 180 degrees
- moved U1088 57.6 mm to (100.9, 87.0), turned to -90 degrees
- moved U1085 52.8 mm to (144.2, 94.2), turned to 180 degrees
- moved D1001 15.0 mm to (114.6, 66.3)
- moved D1013 15.0 mm to (164.7, 57.6), turned to 180 degrees
- moved D1024 15.0 mm to (173.2, 66.4), turned to 90 degrees
- moved D1025 15.0 mm to (173.4, 107.7)
- moved D1012 15.0 mm to (123.4, 57.8), turned to 180 degrees
- moved D1023 10.0 mm to (185.0, 63.8)
- moved D1002 10.0 mm to (102.9, 63.7)
- moved D1014 10.0 mm to (167.3, 45.9)
- moved D1026 10.0 mm to (185.1, 110.3)
- moved D1011 10.00 mm to (120.8, 46.0)
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- renumbered D1002 to D1001, D1003 to D1002, D1004 to D1003, D1005 to D1004, D1006 to D1005, D1007 to D1006, D1008 to D1007, D1009 to D1008, D1010 to D1009, D1011 to D1010, D1012 to D1011, D1013 to D1012, D1015 to D1013, D1016 to D1014, D1017 to D1015, D1018 to D1016, D1019 to D1017, D1020 to D1018, D1021 to D1019, D1022 to D1020, D1023 to D1021, D1024 to D1022, D1025 to D1023, D1026 to D1024, D1028 to D1025, D1029 to D1026, D1030 to D1027, D1031 to D1028, D1032 to D1029, D1033 to D1030, D1034 to D1031, D1035 to D1032, D1036 to D1033, D1037 to D1034, D1038 to D1035, D1039 to D1036, D1041 to D1037, D1042 to D1038, D1043 to D1039, D1044 to D1040, D1045 to D1041, D1046 to D1042, D1047 to D1043, D1048 to D1044, D1049 to D1045, D1050 to D1046, D1051 to D1047, D1052 to D1048
Connections:
- C201 pad 1: Net-(U202-VCC) -> Net-(U202-V3)
- D1001 pad 4: Net-(D1001-DOUT) (its old number) -> Net-(D1001-DIN)
- D1012 pad 2: Net-(D1013-DOUT) (its old number) -> Net-(D1012-DOUT)
- D1013 pad 4: Net-(D1014-DOUT) (its old number) -> Net-(D1012-DOUT)
- D1024 pad 2: Net-(D1026-DOUT) (its old number) -> Net-(D1024-DOUT)
- D1025 pad 4: Net-(D1027-DOUT) (its old number) -> Net-(D1024-DOUT)
- D1036 pad 2: Net-(D1039-DOUT) (its old number) -> Net-(D1036-DOUT)
- D1037 pad 4: Net-(D1040-DOUT) (its old number) -> Net-(D1036-DOUT)
- U202 pad 16: Net-(U202-VCC) -> VBUS
- U202 pad 4: VBUS -> Net-(U202-V3)
Routing:
- net VBUS: track 8.15 -> 160.3 mm
- net +BATT: track 0.00 -> 44.4 mm
- net DTR: track 0.00 -> 10.8 mm
- net Net-(U301-SEL): track 0.00 -> 10.5 mm
- net RTS: track 0.00 -> 9.21 mm
- net Net-(U301-PROG1): track 0.00 -> 8.85 mm
- net Net-(U301-PROG2): track 0.00 -> 8.02 mm
- net Net-(U301-PROG3): track 0.00 -> 6.25 mm
- net Net-(U301-THERM): track 0.00 -> 5.81 mm
- net Net-(U202-V3): track 0.00 -> 4.23 mm
- net Net-(U202-TXD): track 0.00 -> 4.18 mm
- net Net-(U301-~{TE}): track 0.00 -> 4.14 mm
- net Net-(U202-RXD): track 0.00 -> 3.88 mm
- net USB_D+: track 9.24 -> 9.83 mm

Commit message: update
Parts:
- moved C401 168.4 mm to (80.0, 118.3), turned to 90 degrees
- moved U401 155.8 mm to (92.4, 118.3)
- moved R401 149.5 mm to (103.0, 119.5), turned to 90 degrees
- moved R402 144.7 mm to (103.0, 116.0), turned to -90 degrees
- moved R1002 106.7 mm to (157.0, 96.5)
- moved C501 95.8 mm to (156.0, 86.5), turned to 90 degrees
- moved C1085 94.8 mm to (165.9, 83.0)
- moved C502 94.6 mm to (159.5, 86.5), turned to 90 degrees
- moved C1086 93.8 mm to (166.0, 90.0), turned to 0 degrees
- moved R1005 93.8 mm to (157.0, 94.5), turned to 0 degrees
- moved U1086 89.1 mm to (165.9, 86.5), turned to -90 degrees
- moved R501 73.7 mm to (163.0, 75.5), turned to 90 degrees
- moved SW501 69.2 mm to (167.5, 75.3), turned to 90 degrees
- moved LS501 52.9 mm to (209.0, 101.5)
Routing:
- net TP_8: track 0.00 -> 146.1 mm
- net TP_9: track 0.00 -> 145.0 mm
- net TP_7: track 0.00 -> 144.9 mm
- net /Displays/SDA1: track 0.00 -> 132.1 mm
- net TP_5: track 0.00 -> 121.1 mm
- net /Displays/SCL1: track 0.00 -> 119.0 mm
- net TP_6: track 0.00 -> 116.4 mm, vias 0 -> 2
- net TP_4: track 0.00 -> 114.9 mm
- net /Displays/SCL0: track 0.00 -> 107.5 mm
- net /Displays/SDA0: track 0.00 -> 105.1 mm
- net TP_12: track 0.00 -> 95.4 mm
- net TP_11: track 0.00 -> 89.1 mm
- net TP_10: track 0.00 -> 86.4 mm
- net /Displays/IO4: track 0.00 -> 60.3 mm
- net /Displays/IO16: track 0.00 -> 53.5 mm
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
Commit message: update
Parts:
- removed kibuzzard-635B9A1E (x2): G***, kibuzzard-635B9A1E
- removed kibuzzard-635BA762: G***, kibuzzard-635BA762
- removed kibuzzard-635BA7B4: G***, kibuzzard-635BA7B4
- removed kibuzzard-635CF752 (x8): G***, kibuzzard-635CF752
- U1087, U1088, U1089, U1090, U1091: moved to B.Cu
- moved J301 55.1 mm to (141.5, 129.2), turned to 90 degrees
- moved C1085 49.5 mm to (146.0, 128.3), turned to -90 degrees
- moved C301 47.4 mm to (138.2, 141.6), turned to 90 degrees
- moved U1086 45.0 mm to (149.5, 128.3), turned to 0 degrees
- moved BT301 43.0 mm to (176.0, 134.0)
- moved J302 42.4 mm to (141.7, 134.4), turned to 180 degrees
- moved R310 42.1 mm to (141.2, 144.9), turned to -90 degrees
- moved C302 41.6 mm to (141.0, 141.3), turned to 90 degrees
- moved C1086 40.4 mm to (153.0, 128.3), turned to 90 degrees
- moved C303 38.6 mm to (142.9, 137.1), turned to 180 degrees
- moved C304 37.8 mm to (144.2, 147.6), turned to 180 degrees
- moved U301 31.3 mm to (146.2, 142.6), turned to -90 degrees
- moved R302 27.1 mm to (151.7, 149.9), turned to 0 degrees
- moved R301 25.6 mm to (151.7, 133.1), turned to 0 degrees
- moved R305 24.3 mm to (151.7, 147.6), turned to 0 degrees
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Routing:
- net VCC: track 2.36 -> 1162.9 mm
- net +3V3: track 30.5 -> 765.5 mm, vias 0 -> 5
- net Net-(D1087-DOUT): track 0.00 -> 99.5 mm
- net Net-(D1093-DOUT): track 0.00 -> 97.3 mm
- net Net-(D1090-DOUT): track 0.00 -> 95.9 mm
- net /Microcontroller/IO13: track 0.00 -> 70.5 mm
- net /Displays/SDA1: track 132.1 -> 65.2 mm
- net /Displays/SCL1: track 119.0 -> 71.0 mm
- net Net-(D1012-DOUT): track 0.00 -> 44.8 mm
- net Net-(D1036-DOUT): track 0.00 -> 44.6 mm
- net Net-(D1024-DOUT): track 0.00 -> 43.6 mm
- net +BATT: track 44.4 -> 10.2 mm
- net VBUS: track 160.3 -> 127.6 mm
- net /Displays/SCL0: track 107.5 -> 139.5 mm
- net /Displays/IO4: track 60.3 -> 31.6 mm
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Other:
- board text added: "POWER SWITCH"
