File: KiCAD Files/BoardGame/BoardGame.kicad_pcb (KiCad board)
At the start: 2 copper layers, 150 x 150 mm, 131 parts, among them J201 USB_C_Receptacle_USB2.0, J301 Conn_01x01, J302 Conn_01x01, J401 Conn_02x03_Odd_Even, J402 Conn_02x03_Odd_Even, J403 Conn_02x03_Odd_Even, J404 Conn_02x03_Odd_Even, Q1085 UMH3N, SW501 SW_Push, U1085 ESP32-WROOM-32D, U1086 XC6210B332MR, U201 USBLC6-2SC6, U202 CH340C, U301 MCP73871-2CC, U401 PCF8575

Commit message: update
Parts:
- removed R401, R402: 4k7, Resistor_SMD:R_0603_1608Metric
- U1087, U1088, U1089, U1090, U1091: moved to F.Cu
- moved R1002 82.7 mm to (84.5, 108.1), turned to 180 degrees
- moved R1005 55.9 mm to (118.8, 71.0), turned to 180 degrees
- turned U1087 to 0 degrees
- turned U1088 to -90 degrees
- turned U1089 to 180 degrees
- turned U1090 to 90 degrees
- turned U1091 to 0 degrees
Routing:
- net /IO Expander/INT: track 0.00 -> 101.6 mm, vias 0 -> 2
- net /Microcontroller/RESET: track 24.3 -> 117.5 mm, vias 2 -> 12
- net /Microcontroller/IO0: track 0.00 -> 72.2 mm, vias 0 -> 4
- net /Microcontroller/TX: track 0.00 -> 69.4 mm, vias 0 -> 6
- net /Microcontroller/RX: track 0.00 -> 66.6 mm, vias 0 -> 6
- net /Microcontroller/NP_5: track 17.7 -> 77.3 mm, vias 0 -> 4
- net /Microcontroller/NP_2: track 17.2 -> 76.5 mm
- net /Displays/SDA1: track 65.2 -> 114.9 mm, vias 0 -> 2
- net VCC: track 1162.9 -> 1125.5 mm
- net /Displays/SCL1: track 71.0 -> 108.1 mm, vias 0 -> 2
- net /Displays/IO18: track 55.0 -> 25.5 mm, vias 2 -> 0
- net /Displays/IO4: track 31.6 -> 54.4 mm
- net +3V3: track 765.5 -> 744.0 mm, vias 5 -> 3
- net /Displays/IO16: track 29.2 -> 46.1 mm
- net /Displays/IO23: track 32.9 -> 17.2 mm, vias 0 -> 1
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
Commit message: Update BoardGame.kicad_pcb
Routing:
- net GND: vias 148 -> 147
