File: KiCAD Files/BoardGame/BoardGame.kicad_sch (KiCad schematic)
At the start: 0 parts

Commit message: update
Other:
- removed sheet Battery indicator LED
- removed sheet Dice LEDs
- removed sheet Finish LEDs
- removed sheet Safehouse LEDs
- sheet Microcontroller ports: added none; removed NP_1, NP_3, NP_4, NP_6
- note added: "TO-DO: - maknuti ATmega328p i staviti ESP32 - ESP32 autoreset circuit - dodati 3V3 LDO - maknuti 5V boost converter ako se ne koristi - dodati 4x OLED display, 1x okrugli IPS - provjeriti jel sve komponente rade na 3V3"

Commit message: update
Other:
- sheet Boost Converter renamed 3V3 regulator
- sheet Microcontroller ports: added IO0; removed none
- sheet USB ports: added IO0; removed none
Changed lines of the file:
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@@
+	(wire
+		(pts
+			(xy 71.12 66.04) (xy 83.82 66.04)
+		)
+		(stroke
+			(width 0)
+			(type default)
+		)
+	)
 	(wire
 		(pts
@@
 			)
 		)
+		(pin "IO0" input
+			(at 83.82 66.04 180)
+			(effects
+				(font
+					(size 1.27 1.27)
+				)
+				(justify left)
+			)
+		)
 		(instances
 			(project "BoardGame"
@@
 			)
 		)
+		(pin "IO0" output
+			(at 71.12 66.04 0)
+			(effects
+				(font
+					(size 1.27 1.27)
+				)
+				(justify right)
+			)
+		)
 		(instances
 			(project "BoardGame"
@@
 			(color 255 229 191 1.0000)
 		)
-		(property "Sheetname" "Boost Converter"
+		(property "Sheetname" "3V3 regulator"
 			(at 83.82 94.1734 0)
 			(effects

Commit message: update
Other:
- sheet 3V3 regulator renamed 3V3 LDO
- sheet USB renamed USB-UART
- added sheet Displays (Displays.kicad_sch)
- sheet 3V3 LDO ports: added 3V3, VCC; removed none
- sheet Battery charger ports: added VBUS, VCC; removed PG, STAT1, STAT2
- sheet IO Expander ports: added 3V3, SCL0, SDA0; removed SCL, SDA
- sheet Microcontroller ports: added 3V3, IO16, IO17, IO18, IO23, IO4, SCL0, SCL1, SDA0, SDA1; removed PG, SCL, SDA, STAT1, STAT2
- sheet USB-UART ports: added VBUS; removed none
- note added: "TO-DO: - provjeriti jel sve električki točno spojeno - dodijeliti footprinte - TME BOM - bolje razmjestiti rupe da ne zijeva kučište"
- note removed: "TO-DO: - maknuti ATmega328p i staviti ESP32 - ESP32 autoreset circuit - dodati 3V3 LDO - maknuti 5V boost converter ako se ne koristi - dodati 4x OLED display, 1x okrugli IPS - provjeriti jel sve komponente rade na 3V3"

Commit message: update
Other:
- note added: "TO-DO: - provjeriti jel sve električki točno spojeno (isprintati i proči kroz sve) - Nacrtati footprinte koji nedostaju (zasloni) - dodijeliti footprinte - Fixati 3D Modele koji nedostaju na footprintima - TME BOM sastaviti Layout: - bolje razmjestiti rupe da ne zijeva kučište"
- note removed: "TO-DO: - provjeriti jel sve električki točno spojeno - dodijeliti footprinte - TME BOM - bolje razmjestiti rupe da ne zijeva kučište"
Changed lines of the file:
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@@
 		)
 	)
-	(text "TO-DO:\n- provjeriti jel sve električki točno spojeno\n- dodijeliti footprinte\n- TME BOM\n- bolje razmjestiti rupe da ne zijeva kučište"
+	(text "TO-DO:\n- provjeriti jel sve električki točno spojeno (isprintati i proči kroz sve)\n- Nacrtati footprinte koji nedostaju (zasloni)\n- dodijeliti footprinte\n- Fixati 3D Modele koji nedostaju na footprintima\n- TME BOM sastaviti\n\nLayout:\n- bolje razmjestiti rupe da ne zijeva kučište"
 		(exclude_from_sim no)
-		(at 17.78 188.214 0)
+		(at 16.002 184.658 0)
 		(effects
 			(font

Commit message: update
Other:
- note added: "TO-DO: - provjeriti jel sve električki točno spojeno (isprintati i proči kroz sve) - Nacrtati footprinte koji nedostaju (zasloni) - detaljno provjeriti dimenzije - dodijeliti footprinte - Fixati 3D Modele koji nedostaju na footprintima - TME BOM sastaviti Layout: - bolje razmjestiti rupe da ne zijeva kučište"
- note removed: "TO-DO: - provjeriti jel sve električki točno spojeno (isprintati i proči kroz sve) - Nacrtati footprinte koji nedostaju (zasloni) - dodijeliti footprinte - Fixati 3D Modele koji nedostaju na footprintima - TME BOM sastaviti Layout: - bolje razmjestiti rupe da ne zijeva kučište"
Changed lines of the file:
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@@
 		)
 	)
-	(text "TO-DO:\n- provjeriti jel sve električki točno spojeno (isprintati i proči kroz sve)\n- Nacrtati footprinte koji nedostaju (zasloni)\n- dodijeliti footprinte\n- Fixati 3D Modele koji nedostaju na footprintima\n- TME BOM sastaviti\n\nLayout:\n- bolje razmjestiti rupe da ne zijeva kučište"
+	(text "TO-DO:\n- provjeriti jel sve električki točno spojeno (isprintati i proči kroz sve)\n- Nacrtati footprinte koji nedostaju (zasloni) - detaljno provjeriti dimenzije\n- dodijeliti footprinte\n- Fixati 3D Modele koji nedostaju na footprintima\n- TME BOM sastaviti\n\nLayout:\n- bolje razmjestiti rupe da ne zijeva kučište"
 		(exclude_from_sim no)
 		(at 16.002 184.658 0)
@@
 	(sheet
 		(at 73.66 55.88)
-		(size 24.13 22.86)
+		(size 24.13 7.62)
 		(fields_autoplaced yes)
 		(stroke
@@
 		)
 		(property "Sheetfile" "Battery charger.kicad_sch"
-			(at 73.66 79.3246 0)
+			(at 73.66 64.0846 0)
 			(effects
 				(font

Commit message: update
Other:
- note added: "TO-DO: - provjeriti jel sve električki točno spojeno (isprintati i proći kroz sve) - Nacrtati footprinte koji nedostaju (zasloni) - detaljno provjeriti dimenzije - dodijeliti footprinte - Fixati 3D Modele koji nedostaju na footprintima - TME BOM sastaviti Layout: - bolje razmjestiti rupe da ne zijeva kučište"
- note removed: "TO-DO: - provjeriti jel sve električki točno spojeno (isprintati i proči kroz sve) - Nacrtati footprinte koji nedostaju (zasloni) - detaljno provjeriti dimenzije - dodijeliti footprinte - Fixati 3D Modele koji nedostaju na footprintima - TME BOM sastaviti Layout: - bolje razmjestiti rupe da ne zijeva kučište"
Changed lines of the file:
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@@
 		)
 	)
-	(text "TO-DO:\n- provjeriti jel sve električki točno spojeno (isprintati i proči kroz sve)\n- Nacrtati footprinte koji nedostaju (zasloni) - detaljno provjeriti dimenzije\n- dodijeliti footprinte\n- Fixati 3D Modele koji nedostaju na footprintima\n- TME BOM sastaviti\n\nLayout:\n- bolje razmjestiti rupe da ne zijeva kučište"
+	(text "TO-DO:\n- provjeriti jel sve električki točno spojeno (isprintati i proći kroz sve)\n- Nacrtati footprinte koji nedostaju (zasloni) - detaljno provjeriti dimenzije\n- dodijeliti footprinte\n- Fixati 3D Modele koji nedostaju na footprintima\n- TME BOM sastaviti\n\nLayout:\n- bolje razmjestiti rupe da ne zijeva kučište"
 		(exclude_from_sim no)
 		(at 16.002 184.658 0)

Commit message: update
Other:
- note added: "TO-DO: - ispraviti dimenzije baterije - pomaknuti bateriju na bolju poziciju - provjeriti poziciju buzzera - premjestiti pinove da bolje odgovaraju layoutu (testirati na breadboardu) - provjeriti jel sve električki točno spojeno (isprintati i proći kroz sve) - Nacrtati footprinte koji nedostaju (zasloni) - detaljno provjeriti dimenzije - dodijeliti footprinte - Fixati 3D Modele koji nedostaju na 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"
- note removed: "TO-DO: - provjeriti jel sve električki točno spojeno (isprintati i proći kroz sve) - Nacrtati footprinte koji nedostaju (zasloni) - detaljno provjeriti dimenzije - dodijeliti footprinte - Fixati 3D Modele koji nedostaju na footprintima - TME BOM sastaviti Layout: - bolje razmjestiti rupe da ne zijeva kučište"
Changed lines of the file:
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@@
 		)
 	)
-	(text "TO-DO:\n- provjeriti jel sve električki točno spojeno (isprintati i proći kroz sve)\n- Nacrtati footprinte koji nedostaju (zasloni) - detaljno provjeriti dimenzije\n- dodijeliti footprinte\n- Fixati 3D Modele koji nedostaju na footprintima\n- TME BOM sastaviti\n\nLayout:\n- bolje razmjestiti rupe da ne zijeva kučište"
+	(text "TO-DO:\n- ispraviti dimenzije baterije\n- pomaknuti bateriju na bolju poziciju\n- provjeriti poziciju buzzera\n- premjestiti pinove da bolje odgovaraju layoutu (testirati na breadboardu)\n- provjeriti jel sve električki točno spojeno (isprintati i proći kroz sve)\n- Nacrtati footprinte koji nedostaju (zasloni) - detaljno provjeriti dimenzije\n- dodijeliti footprinte\n- Fixati 3D Modele koji nedostaju na footprintima\n- TME BOM sastaviti\n\nLayout:\n- bolje razmjestiti rupe da ne zijeva kučište"
 		(exclude_from_sim no)
 		(at 16.002 184.658 0)

Commit message: update
Other:
- note added: "TO-DO: - dodati 3D model baterije, debljina je 6mm - centrirati MCU na sredinu pločice - pomaknuti bateriju na bolju poziciju - provjeriti poziciju buzzera - premjestiti pinove da bolje odgovaraju layoutu (testirati na breadboardu) - provjeriti jel sve električki točno spojeno (isprintati i proći kroz sve) - Nacrtati footprinte koji nedostaju (zasloni) - detaljno provjeriti dimenzije - dodijeliti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"
- note removed: "TO-DO: - ispraviti dimenzije baterije - pomaknuti bateriju na bolju poziciju - provjeriti poziciju buzzera - premjestiti pinove da bolje odgovaraju layoutu (testirati na breadboardu) - provjeriti jel sve električki točno spojeno (isprintati i proći kroz sve) - Nacrtati footprinte koji nedostaju (zasloni) - detaljno provjeriti dimenzije - dodijeliti footprinte - Fixati 3D Modele koji nedostaju na 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"
Changed lines of the file:
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@@
 		)
 	)
-	(text "TO-DO:\n- ispraviti dimenzije baterije\n- pomaknuti bateriju na bolju poziciju\n- provjeriti poziciju buzzera\n- premjestiti pinove da bolje odgovaraju layoutu (testirati na breadboardu)\n- provjeriti jel sve električki točno spojeno (isprintati i proći kroz sve)\n- Nacrtati footprinte koji nedostaju (zasloni) - detaljno provjeriti dimenzije\n- dodijeliti footprinte\n- Fixati 3D Modele koji nedostaju na footprintima\n- TME BOM sastaviti\n\nLayout:\n- bolje razmjestiti rupe da ne zijeva kučište"
+	(text "TO-DO:\n- dodati 3D model baterije, debljina je 6mm\n- centrirati MCU na sredinu pločice\n- pomaknuti bateriju na bolju poziciju\n- provjeriti poziciju buzzera\n- premjestiti pinove da bolje odgovaraju layoutu (testirati na breadboardu)\n- provjeriti jel sve električki točno spojeno (isprintati i proći kroz sve)\n- Nacrtati footprinte koji nedostaju (zasloni) - detaljno provjeriti dimenzije\n- dodijeliti footprinte\n- Fixati 3D Modele koji nedostaju na footprintima\n- TME BOM sastaviti\n\nLayout:\n- bolje razmjestiti rupe da ne zijeva kučište"
 		(exclude_from_sim no)
 		(at 16.002 184.658 0)
