File: KiCAD Files/BoardGame/BoardGame.kicad_sch (KiCad schematic)
At the start: 0 parts

Commit message: update
Other:
- note added: "TO-DO: - provjeriti jel sve električki točno spojeno (isprintati i proći kroz sve) - Fixati 3D Modele koji nedostaju na footprintima - Assembly svega + nova gornja površina tematski ukrašena - TME BOM sastaviti - pored ovoga, na izradu poslati još i CNLJS (ploča + kockica + TP) Layout: - bolje razmjestiti rupe da ne zijeva kučište"
- note removed: "TO-DO: - provjeriti odgovaraju li dimenzije svih zaslona - provjeriti jel sve električki točno spojeno (isprintati i proći kroz sve) - Nacrtati footprinte koji nedostaju (zasloni) - detaljno provjeriti dimenzije - dodijeliti footprinte - Fixati 3D Modele koji nedostaju na footprintima - TME BOM sastaviti - pored ovoga, na izradu poslati još i CNLJS (ploča + kockica + TP) Layout: - bolje razmjesti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"
Changed lines of the file:
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@@
 		)
 	)
-	(text "TO-DO:\n- provjeriti odgovaraju li dimenzije svih zaslona\n- provjeriti jel sve električki točno spojeno (isprintati i proći kroz sve)\n- Nacrtati footprinte koji nedostaju (zasloni) - detaljno provjeriti dimenzije\n- dodijeliti footprinte\n- Fixati 3D Modele koji nedostaju na footprintima\n- TME BOM sastaviti\n- pored ovoga, na izradu poslati još i CNLJS (ploča + kockica + TP)\n\nLayout:\n- bolje razmjestiti rupe da ne zijeva kučište"
+	(text "TO-DO:\n- provjeriti jel sve električki točno spojeno (isprintati i proći kroz sve)\n- Fixati 3D Modele koji nedostaju na footprintima\n- Assembly svega + nova gornja površina tematski ukrašena\n- TME BOM sastaviti\n- pored ovoga, na izradu poslati još i CNLJS (ploča + kockica + TP)\n\nLayout:\n- bolje razmjestiti rupe da ne zijeva kučište"
 		(exclude_from_sim no)
 		(at 16.002 180.848 0)

Commit message: update
Other:
- note added: "TO-DO: - Assembly svega + nova gornja površina tematski ukrašena"
- note removed: "TO-DO: - provjeriti jel sve električki točno spojeno (isprintati i proći kroz sve) - Fixati 3D Modele koji nedostaju na footprintima - Assembly svega + nova gornja površina tematski ukrašena - TME BOM sastaviti - pored ovoga, na izradu poslati još i CNLJS (ploča + kockica + TP) Layout: - bolje razmjestiti rupe da ne zijeva kučište"
Changed lines of the file:
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@@
 		)
 	)
-	(text "TO-DO:\n- provjeriti jel sve električki točno spojeno (isprintati i proći kroz sve)\n- Fixati 3D Modele koji nedostaju na footprintima\n- Assembly svega + nova gornja površina tematski ukrašena\n- TME BOM sastaviti\n- pored ovoga, na izradu poslati još i CNLJS (ploča + kockica + TP)\n\nLayout:\n- bolje razmjestiti rupe da ne zijeva kučište"
+	(text "TO-DO:\n- Assembly svega + nova gornja površina tematski ukrašena"
 		(exclude_from_sim no)
 		(at 16.002 180.848 0)
