File: KiCAD Files/BoardGame/IO Expander.kicad_sch (KiCad schematic)
At the start: 12 parts, among them J401 Conn_02x03_Odd_Even, J402 Conn_02x03_Odd_Even, J403 Conn_02x03_Odd_Even, J404 Conn_02x03_Odd_Even, J405 Conn_01x02_Female, J406 Conn_01x02_Female, J407 Conn_01x02_Female, J408 Conn_01x02_Female, U401 PCF8575

Commit message: update
Parts:
- removed J405, J406, J407, J408: Conn_01x02_Female, Connector_PinHeader_1.27mm:PinHeader_1x02_P1.27mm_Vertical, symbol Connector:Conn_01x02_Female
Connections:
- net +5V renamed +3V3
- no-connect marks 8 -> 6
Other:
- note removed: "Dice touchpad connectors"
- moved on the sheet: J401, J402, J403, J404

Commit message: update
Connections:
- net SCL renamed SCL0
- net SDA renamed SDA0
- net TP_13: no longer names the net of U401.17 (P14)
- no-connect marks 6 -> 7
Changed lines of the file:
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@@
 		(at 76.2 90.17)
 	)
+	(no_connect
+		(at 96.52 100.33)
+	)
 	(wire
 		(pts
@@
 		(pts
 			(xy 184.15 102.87) (xy 173.99 102.87)
+		)
+		(stroke
+			(width 0)
+			(type default)
+		)
+	)
+	(wire
+		(pts
+			(xy 31.75 64.77) (xy 31.75 66.04)
 		)
 		(stroke
@@
 		)
 	)
-	(global_label "TP_13"
-		(shape input)
-		(at 96.52 100.33 0)
-		(fields_autoplaced yes)
-		(effects
-			(font
-				(size 1.27 1.27)
-			)
-			(justify left)
-		)
-		(property "Intersheetrefs" "${INTERSHEET_REFS}"
-			(at 104.5574 100.2506 0)
-			(effects
-				(font
-					(size 1.27 1.27)
-				)
-				(justify left)
-				(hide yes)
-			)
-		)
-	)
 	(global_label "TP_8"
 		(shape input)
@@
 		)
 	)
-	(hierarchical_label "SDA"
+	(hierarchical_label "3V3"
+		(shape input)
+		(at 31.75 66.04 270)
+		(fields_autoplaced yes)
+		(effects
+			(font
+				(size 1.27 1.27)
+			)
+			(justify right)
+		)
+	)
+	(hierarchical_label "SDA0"
 		(shape bidirectional)
 		(at 59.69 107.95 180)
@@
 		)
 	)
-	(hierarchical_label "SCL"
+	(hierarchical_label "SCL0"
 		(shape input)
 		(at 59.69 105.41 180)
@@
 			)
 		)
-		(property "Description" ""
+		(property "Description" "Power symbol creates a global label with name \"GND\" , ground"
 			(at 152.4 82.55 0)
 			(effects
@@
 	)
 	(symbol
+		(lib_id "power:+3V3")
+		(at 31.75 64.77 0)
+		(unit 1)
+		(exclude_from_sim no)
+		(in_bom yes)
+		(on_board yes)
+		(dnp no)
+		(fields_autoplaced yes)
+		(property "Reference" "#PWR01126"
+			(at 31.75 68.58 0)
+			(effects
+				(font
+					(size 1.27 1.27)
+				)
+				(hide yes)
+			)
+		)
+		(property "Value" "+3V3"
+			(at 31.75 59.69 0)
+			(effects
+				(font
+					(size 1.27 1.27)
+				)
+			)
+		)
+		(property "Footprint" ""
+			(at 31.75 64.77 0)
+			(effects
+				(font
+					(size 1.27 1.27)
+				)
+				(hide yes)
+			)
+		)
+		(property "Datasheet" ""
+			(at 31.75 64.77 0)
+			(effects
+				(font
+					(size 1.27 1.27)
+				)
+				(hide yes)
+			)
+		)
+		(property "Description" "Power symbol creates a global label with name \"+3V3\""
+			(at 31.75 64.77 0)
+			(effects
+				(font
+					(size 1.27 1.27)
+				)
+				(hide yes)
+			)
+		)
+		(pin "1"
+		)
+		(instances
+			(project ""
+				(path "/9f66d68b-38d2-4517-8629-387431399ae9/defa6cf4-007a-48e8-ac65-029b900cd1cd"
+					(reference "#PWR01126")
+					(unit 1)
+				)
+			)
+		)
+	)
+	(symbol
 		(lib_id "Connector_Generic:Conn_02x03_Odd_Even")
 		(at 166.37 102.87 0)
@@
 			)
 		)
-		(property "Description" ""
+		(property "Description" "Power symbol creates a global label with name \"GND\" , ground"
 			(at 152.4 130.81 0)
 			(effects
@@
 			)
 		)
-		(property "Description" ""
+		(property "Description" "Power symbol creates a global label with name \"GND\" , ground"
 			(at 152.4 59.69 0)
 			(effects
@@
 			)
 		)
-		(property "Description" ""
+		(property "Description" "Power symbol creates a global label with name \"GND\" , ground"
 			(at 86.36 113.03 0)
 			(effects
@@
 			)
 		)
-		(property "Description" ""
+		(property "Description" "Power symbol creates a global label with name \"GND\" , ground"
 			(at 59.69 72.39 0)
 			(effects
@@
 			)
 		)
-		(property "Description" ""
+		(property "Description" "Power symbol creates a global label with name \"GND\" , ground"
 			(at 152.4 107.95 0)
 			(effects

Commit message: update
Parts:
- removed R401, R402: 4k7, Resistor_SMD:R_0603_1608Metric, symbol Device:R_Small
