File: KiCAD Files/PushButtons/PushButtons.kicad_pcb (KiCad board)
At the start: 2 copper layers, 88.5 x 30 mm, 8 parts, among them J1 Conn_01x04_Pin, SW1 SW_Push, SW2 SW_Push, SW3 SW_Push

Commit message: update
Parts:
- removed J1: Conn_01x04_Pin, Connector_PinHeader_2.54mm:PinHeader_1x04_P2.54mm_Horizontal
- added D1: WS2812B, LED_SMD:LED_WS2812B_PLCC4_5.0x5.0mm_P3.2mm, F.Cu at (80.8, 32.5)
- added D2: WS2812B, LED_SMD:LED_WS2812B_PLCC4_5.0x5.0mm_P3.2mm, F.Cu at (97.0, 32.5)
- added D3: WS2812B, LED_SMD:LED_WS2812B_PLCC4_5.0x5.0mm_P3.2mm, F.Cu at (108.0, 32.5)
- added D4: WS2812B, LED_SMD:LED_WS2812B_PLCC4_5.0x5.0mm_P3.2mm, F.Cu at (119.5, 32.5)
Other:
- board size 88.5 x 30 mm -> 76.8 x 30 mm

Commit message: update
Parts:
- added J1: Conn_01x07_Pin, Connector_PinHeader_2.54mm:PinHeader_1x07_P2.54mm_Horizontal, B.Cu at (109.1, 42.5)
- moved D4 5.95 mm to (125.5, 32.5), turned to 180 degrees
- moved D2 3.55 mm to (93.5, 32.5), turned to 180 degrees
- moved D1 3.30 mm to (77.5, 32.5), turned to 180 degrees
- moved D3 1.45 mm to (109.5, 32.5), turned to 180 degrees
Routing:
- net /VCC: track 0.00 -> 66.7 mm
- net /DOUT: track 0.00 -> 43.2 mm, vias 0 -> 1
- net /B1: track 0.00 -> 28.1 mm
- net /DIN: track 0.00 -> 27.5 mm
- net /B3: track 0.00 -> 19.2 mm
- net Net-(D3-DOUT): track 0.00 -> 12.5 mm
- net Net-(D2-DOUT): track 0.00 -> 12.5 mm
- net Net-(D1-DOUT): track 0.00 -> 12.5 mm
- net /B2: track 0.00 -> 10.8 mm
- added copper zone on B.Cu, net /GND
- added copper zone on F.Cu, net /GND
Other:
- board text added: "B1"
- board text added: "B2"
- board text added: "B3"
- board text added: "DIN"
- board text added: "DOUT"
- board text added: "GND"
- board text added: "VCC"
