File: KiCAD Files/FullPCB/FullPCB.kicad_pcb (KiCad board)
At the start: 2 copper layers, 172.1 x 172.1 mm, 40 parts, among them J1 OLED1, J2 OLED2, J3 OLED3, J4 OLED4, J5 Conn_01x08, SW1 SW_Push_Dual, SW10 SW_Push_Dual, SW11 SW_Push_Dual, SW12 SW_Push_Dual, SW2 SW_Push_Dual, SW3 SW_Push_Dual, SW4 SW_Push_Dual, SW5 SW_Push_Dual, SW6 SW_Push_Dual, SW7 SW_Push_Dual, SW8 SW_Push_Dual, SW9 SW_Push_Dual

Commit message: update
Parts:
- removed J3: OLED3, Connector_PinHeader_2.54mm:PinHeader_1x04_P2.54mm_Horizontal
- removed J4: OLED4, Connector_PinHeader_2.54mm:PinHeader_1x04_P2.54mm_Horizontal
- J1: value OLED1 -> OLED1&2; footprint Connector_PinHeader_2.54mm:PinHeader_1x04_P2.54mm_Horizontal -> Library:JST_SH_SM04B-SRSS-TB_1x04-1MP_P1.00mm; moved to B.Cu
- J2: value OLED2 -> OLED3&4; footprint Connector_PinHeader_2.54mm:PinHeader_1x04_P2.54mm_Horizontal -> Library:JST_SH_SM04B-SRSS-TB_1x04-1MP_P1.00mm; moved to B.Cu
- moved J5 96.3 mm to (135.4, 93.7), turned to -135 degrees
- moved J2 92.7 mm to (120.5, 88.5), turned to 135 degrees
- moved J1 91.2 mm to (128.8, 96.7), turned to 135 degrees
- moved R2 0.35 mm to (141.1, 64.8)
- moved R4 0.30 mm to (134.0, 72.0)
Connections:
- J2 pad 1: /I2C1_SCL -> /I2C2_SCL
- J2 pad 2: /I2C1_SDA -> /I2C2_SDA
Routing:
- net +5V: track 0.00 -> 562.2 mm
- net /B5: track 6.50 -> 256.8 mm, vias 0 -> 2
- net /B2: track 6.50 -> 210.2 mm, vias 0 -> 2
- net /B1: track 6.50 -> 182.7 mm, vias 0 -> 2
- net /B3: track 6.50 -> 181.5 mm
- net /B4: track 6.50 -> 179.0 mm, vias 0 -> 4
- net /B6: track 6.50 -> 160.8 mm, vias 0 -> 1
- net /B10: track 6.50 -> 100.9 mm, vias 0 -> 2
- net /B11: track 6.50 -> 94.0 mm
- net /RST: track 0.00 -> 84.4 mm
- net /CS: track 0.00 -> 79.3 mm
- net /B12: track 6.50 -> 85.5 mm
- net +3.3V: track 0.00 -> 73.7 mm
- net /DC: track 0.00 -> 73.5 mm
- net /B9: track 6.50 -> 71.6 mm
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Other:
- outline, holes or cut-outs redrawn
- board text added: "BLK"
- board text added: "CS"
- board text added: "DC"
- board text added: "DUMMY"
- board text added: "GND"
- board text added: "J1"
- board text added: "J2"
- board text added: "RST"
- board text added: "SCL"
- board text added: "SDA"
- board text added: "SW1"
- board text added: "SW10"
- board text added: "SW11"
- board text added: "SW12"
- board text added: "SW2"
- board text added: "SW3"
- board text added: "SW4"
- board text added: "SW5"
- board text added: "SW6"
- board text added: "SW7"
- board text added: "SW8"
- board text added: "SW9"
- board text added: "VCC"

Commit message: update
Connections:
- J1 pad 1: /I2C1_SCL -> GND
- J1 pad 2: /I2C1_SDA -> +3.3V
- J1 pad 3: +3.3V -> /I2C1_SDA
- J1 pad 4: GND -> /I2C1_SCL
- J2 pad 1: /I2C2_SCL -> GND
- J2 pad 2: /I2C2_SDA -> +3.3V
- J2 pad 3: +3.3V -> /I2C2_SDA
- J2 pad 4: GND -> /I2C2_SCL
Routing:
- net /I2C2_SCL: track 37.0 -> 29.5 mm
- net /I2C1_SCL: track 29.6 -> 36.7 mm
- net /I2C1_SDA: track 31.8 -> 37.4 mm
- net GND: vias 4 -> 5
Changed lines of the file:
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@@
 			(layers "B.Cu" "B.Mask" "B.Paste")
 			(roundrect_rratio 0.25)
-			(net 21 "/I2C1_SCL")
+			(net 25 "GND")
 			(pinfunction "Pin_1")
 			(pintype "passive")
@@
 			(layers "B.Cu" "B.Mask" "B.Paste")
 			(roundrect_rratio 0.25)
-			(net 46 "/I2C1_SDA")
+			(net 2 "+3.3V")
 			(pinfunction "Pin_2")
 			(pintype "passive")
@@
 			(layers "B.Cu" "B.Mask" "B.Paste")
 			(roundrect_rratio 0.25)
-			(net 2 "+3.3V")
+			(net 46 "/I2C1_SDA")
 			(pinfunction "Pin_3")
 			(pintype "passive")
@@
 			(layers "B.Cu" "B.Mask" "B.Paste")
 			(roundrect_rratio 0.25)
-			(net 25 "GND")
+			(net 21 "/I2C1_SCL")
 			(pinfunction "Pin_4")
 			(pintype "passive")
@@
 			(layers "B.Cu" "B.Mask" "B.Paste")
 			(roundrect_rratio 0.25)
-			(net 17 "/I2C2_SCL")
+			(net 25 "GND")
 			(pinfunction "Pin_1")
 			(pintype "passive")
@@
 			(layers "B.Cu" "B.Mask" "B.Paste")
 			(roundrect_rratio 0.25)
-			(net 23 "/I2C2_SDA")
+			(net 2 "+3.3V")
 			(pinfunction "Pin_2")
 			(pintype "passive")
@@
 			(layers "B.Cu" "B.Mask" "B.Paste")
 			(roundrect_rratio 0.25)
-			(net 2 "+3.3V")
+			(net 23 "/I2C2_SDA")
 			(pinfunction "Pin_3")
 			(pintype "passive")
@@
 			(layers "B.Cu" "B.Mask" "B.Paste")
 			(roundrect_rratio 0.25)
-			(net 25 "GND")
+			(net 17 "/I2C2_SCL")
 			(pinfunction "Pin_4")
 			(pintype "passive")
@@
 	)
 	(segment
-		(start 122.998532 84.5)
-		(end 124.592858 82.905674)
-		(width 0.5)
+		(start 124.592858 82.905674)
+		(end 127.326216 80.172316)
+		(width 1)
 		(layer "B.Cu")
 		(net 2)
 	)
 	(segment
-		(start 121.56066 86.732233)
-		(end 122.998532 85.294361)
+		(start 134.551146 94.5)
+		(end 131.666905 94.5)
 		(width 0.5)
 		(layer "B.Cu")
@@
 	)
 	(segment
-		(start 125.5 81.998532)
-		(end 125.5 79.5)
-		(width 1)
+		(start 123.5 86.207107)
+		(end 122.267767 87.43934)
+		(width 0.5)
 		(layer "B.Cu")
 		(net 2)
 	)
 	(segment
-		(start 135.369165 93.681981)
-		(end 131.07071 93.681981)
-		(width 0.5)
+		(start 127.326216 80.172316)
+		(end 127.326216 72.576162)
+		(width 1)
 		(layer "B.Cu")
 		(net 2)
 	)
 	(segment
-		(start 125.5 79.5)
-		(end 127.326216 77.673784)
-		(width 1)
+		(start 123.5 84)
+		(end 123.5 86.207107)
+		(width 0.5)
 		(layer "B.Cu")
 		(net 2)
 	)
 	(segment
-		(start 131.07071 93.681981)
-		(end 129.866384 94.886307)
+		(start 135.369165 93.681981)
+		(end 134.551146 94.5)
 		(width 0.5)
 		(layer "B.Cu")
@@
 	)
 	(segment
-		(start 122.998532 85.294361)
-		(end 122.998532 84.5)
+		(start 124.592858 82.905674)
+		(end 124.592858 82.907142)
 		(width 0.5)
 		(layer "B.Cu")
@@
 	)
 	(segment
-		(start 124.592858 82.905674)
-		(end 125.5 81.998532)
-		(width 1)
+		(start 124.592858 82.907142)
+		(end 123.5 84)
+		(width 0.5)
 		(layer "B.Cu")
 		(net 2)
 	)
 	(segment
-		(start 127.326216 77.673784)
-		(end 127.326216 72.576162)
-		(width 1)
+		(start 131.666905 94.5)
+		(end 130.573491 95.593414)
+		(width 0.5)
 		(layer "B.Cu")
 		(net 2)
@@
 	)
 	(segment
-		(start 131.5 64.5)
-		(end 118.5 77.5)
-		(width 0.2)
-		(layer "B.Cu")
-		(net 17)
-	)
-	(segment
-		(start 122.121321 89)
-		(end 122.974874 88.146447)
-		(width 0.2)
-		(layer "B.Cu")
-		(net 17)
-	)
-	(segment
-		(start 134.545776 65.427312)
-		(end 133.618464 64.5)
+		(start 119 78)
+		(end 131.572688 65.427312)
 		(width 0.2)
 		(layer "B.Cu")
@@
 	)
 	(segment
-		(start 133.618464 64.5)
-		(end 131.5 64.5)
+		(start 131.572688 65.427312)
+		(end 134.545776 65.427312)
 		(width 0.2)
 		(layer "B.Cu")
@@
 	)
 	(segment
-		(start 120.5 89)
-		(end 122.121321 89)
+		(start 119 84.171573)
+		(end 119 78)
 		(width 0.2)
 		(layer "B.Cu")
@@
 	)
 	(segment
-		(start 118.5 77.5)
-		(end 118.5 87)
-		(width 0.2)
-		(layer "B.Cu")
-		(net 17)
-	)
-	(segment
-		(start 118.5 87)
-		(end 120.5 89)
+		(start 120.853553 86.025126)
+		(end 119 84.171573)
 		(width 0.2)
 		(layer "B.Cu")
@@
 	)
 	(segment
-		(start 150.809232 86.190768)
-		(end 150.809232 81.690768)
+		(start 150.809232 81.690768)
+		(end 150.809232 85.190768)
+		(width 0.2)
+		(layer "B.Cu")
+		(net 21)
+	)
+	(segment
+		(start 128 95.338478)
+		(end 129.159278 94.1792)
 		(width 0.2)
 		(layer "B.Cu")
@@
 	)
 	(segment
-		(start 131.280598 96.300521)
-		(end 132.980077 98)
+		(start 131.5 100)
+		(end 128 96.5)
 		(width 0.2)
 		(layer "B.Cu")
@@
 	)
 	(segment
-		(start 139 98)
-		(end 150.809232 86.190768)
+		(start 150.809232 85.190768)
+		(end 136 100)
 		(width 0.2)
 		(layer "B.Cu")
@@
 	)
 	(segment
-		(start 132.980077 98)
-		(end 139 98)
+		(start 128 96.5)
+		(end 128 95.338478)
+		(width 0.2)
+		(layer "B.Cu")
+		(net 21)
+	)
+	(segment
+		(start 136 100)
+		(end 131.5 100)
 		(width 0.2)
 		(layer "B.Cu")
@@
 	)
 	(segment
-		(start 136.341827 66.158173)
-		(end 135.5 67)
+		(start 117.5 78)
+		(end 117.5 85.5)
 		(width 0.2)
 		(layer "B.Cu")
@@
 	)
 	(segment
-		(start 131.5 66)
-		(end 119.5 78)
-		(width 0.2)
-		(layer "B.Cu")
-		(net 23)
-	)
-	(segment
-		(start 119.5 78)
-		(end 119.5 87)
+		(start 117.5 85.5)
+		(end 119.5 87.5)
 		(width 0.2)
 		(layer "B.Cu")
@@
 	(segment
 		(start 136.341827 63.631261)
-		(end 136.341827 66.158173)
-		(width 0.2)
-		(layer "B.Cu")
-		(net 23)
-	)
-	(segment
-		(start 120.5 88)
-		(end 121.707107 88)
-		(width 0.2)
-		(layer "B.Cu")
-		(net 23)
-	)
-	(segment
-		(start 121.707107 88)
-		(end 122.267767 87.43934)
+		(end 131.868739 63.631261)
 		(width 0.2)
 		(layer "B.Cu")
@@
 	)
 	(segment
-		(start 134.25 67)
-		(end 133.25 66)
-		(width 0.2)
-		(layer "B.Cu")
-		(net 23)
-	)
-	(segment
-		(start 133.25 66)
-		(end 131.5 66)
+		(start 121.56066 86.732233)
+		(end 120.792893 87.5)
 		(width 0.2)
 		(layer "B.Cu")
@@
 	)
 	(segment
-		(start 119.5 87)
-		(end 120.5 88)
+		(start 119.5 87.5)
+		(end 120.792893 87.5)
 		(width 0.2)
 		(layer "B.Cu")
@@
 	)
 	(segment
-		(start 135.5 67)
-		(end 134.25 67)
+		(start 131.868739 63.631261)
+		(end 117.5 78)
 		(width 0.2)
 		(layer "B.Cu")
@@
 	)
 	(via
-		(at 130 93)
+		(at 132.5 98)
 		(size 0.6)
 		(drill 0.3)
@@
 	)
 	(via
-		(at 121.9 84.4)
+		(at 122.75 89.75)
 		(size 0.6)
 		(drill 0.3)
@@
 	)
 	(via
+		(at 121.75 83.25)
+		(size 0.6)
+		(drill 0.3)
+		(layers "F.Cu" "B.Cu")
+		(free yes)
+		(net 25)
+	)
+	(via
 		(at 175.5 115)
 		(size 0.6)
@@
 	)
 	(segment
-		(start 138 94)
-		(end 138 90)
+		(start 141 93.5)
+		(end 141 88)
 		(width 0.2)
 		(layer "B.Cu")
@@
 	)
 	(segment
-		(start 136 96)
-		(end 138 94)
+		(start 131.75 99)
+		(end 135.5 99)
 		(width 0.2)
 		(layer "B.Cu")
@@
 	)
 	(segment
-		(start 131.232981 94.933924)
-		(end 132.933924 94.933924)
+		(start 129.866384 94.886307)
+		(end 129.25 95.502691)
 		(width 0.2)
 		(layer "B.Cu")
@@
 	)
 	(segment
-		(start 148.105283 79.894717)
+		(start 149.105283 79.894717)
 		(end 152.605283 79.894717)
 		(width 0.2)
@@
 	)
 	(segment
-		(start 132.933924 94.933924)
-		(end 134 96)
+		(start 129.25 96.5)
+		(end 131.75 99)
 		(width 0.2)
 		(layer "B.Cu")
@@
 	)
 	(segment
-		(start 134 96)
-		(end 136 96)
+		(start 135.5 99)
+		(end 141 93.5)
 		(width 0.2)
 		(layer "B.Cu")
@@
 	)
 	(segment
-		(start 138 90)
-		(end 148.105283 79.894717)
+		(start 129.25 95.502691)
+		(end 129.25 96.5)
 		(width 0.2)
 		(layer "B.Cu")
@@
 	)
 	(segment
-		(start 130.573491 95.593414)
-		(end 131.232981 94.933924)
+		(start 141 88)
+		(end 149.105283 79.894717)
 		(width 0.2)
 		(layer "B.Cu")
