File: KiCAD Files/FarmGameV2/FarmGameV2.kicad_pcb (KiCad board)
At the start: 2 copper layers, 172.1 x 172.1 mm, 38 parts, among them J1 OLED1&2, J2 OLED3&4, J5 Conn_01x08, SW1 SW_Push_Dual, SW10 SW_Push_Dual, SW11 SW_Push_Dual, SW12 SW_Push_Dual, SW2 SW_Push_Dual, SW3 SW_Push_Dual, SW4 SW_Push_Dual, SW5 SW_Push_Dual, SW6 SW_Push_Dual, SW7 SW_Push_Dual, SW8 SW_Push_Dual, SW9 SW_Push_Dual

Commit message: update
Parts:
- removed J1: OLED1&2, Library:JST_SH_SM04B-SRSS-TB_1x04-1MP_P1.00mm
- removed U1: ~, Library:LOLIN32
- added BZ1: Buzzer, Buzzer_Beeper:Buzzer_TDK_PS1240P02BT_D12.2mm_H6.5mm, F.Cu at (248.6, 104.3)
- added Q1: MMBT2222A, Package_TO_SOT_SMD:SOT-23, F.Cu at (260.4, 99.7)
- added Q2: BC847, Package_TO_SOT_SMD:SOT-23, F.Cu at (260.4, 104.1)
- added Q3: AO3401A, Package_TO_SOT_SMD:SOT-23, F.Cu at (260.4, 108.5)
- added R6: 100R, Resistor_SMD:R_0805_2012Metric, F.Cu at (241.8, 110.7)
- added SW13: POWER, Connector_PinHeader_2.54mm:PinHeader_1x02_P2.54mm_Vertical, F.Cu at (224.0, 43.5)
- added U2: ~, Library:ESP32-S3, B.Cu at (220.7, 52.5)
- added U3: ~, Library:PCF8575, F.Cu at (249.0, 76.5)
- R3, R5: value 10k -> 1k
- moved R4 112.7 mm to (241.8, 104.8), turned to 0 degrees
- moved R5 111.8 mm to (241.8, 107.8), turned to 0 degrees
- moved R2 106.2 mm to (241.8, 98.9), turned to 0 degrees
- moved R3 105.7 mm to (241.8, 101.8), turned to 0 degrees
Connections:
- net +5V renamed VCC
- R2 pad 1: /B9 -> +BATT
- R2 pad 2: +3.3V -> Net-(Q2-C)
- R3 pad 1: /B10 -> /EN
- R3 pad 2: +3.3V -> Net-(Q2-B)
- R4 pad 1: /B11 -> Net-(Q2-B)
- R4 pad 2: +3.3V -> GND
- R5 pad 1: /B12 -> Net-(Q2-C)
- R5 pad 2: +3.3V -> Net-(Q3-G)
Routing:
- net VCC: track 562.2 -> 0.00 mm
- net /B5: track 256.8 -> 0.00 mm, vias 2 -> 0
- net /B2: track 210.2 -> 0.00 mm, vias 2 -> 0
- net Net-(D13-DOUT): track 195.2 -> 0.00 mm
- net Net-(D10-DIN): track 190.3 -> 0.00 mm
- net Net-(D5-DOUT): track 183.3 -> 0.00 mm
- net /B1: track 182.7 -> 0.00 mm, vias 2 -> 0
- net /B3: track 181.5 -> 0.00 mm
- net /B4: track 179.0 -> 0.00 mm, vias 4 -> 0
- net Net-(D1-DIN): track 174.5 -> 0.00 mm
- net /B6: track 160.8 -> 0.00 mm, vias 1 -> 0
- net /B10: track 100.9 -> 0.00 mm, vias 2 -> 0
- net /B11: track 94.0 -> 0.00 mm
- net /B12: track 85.5 -> 0.00 mm
- net /RST: track 84.4 -> 0.00 mm
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
Commit message: update
Parts:
- added R10: 10k, Resistor_SMD:R_0805_2012Metric, B.Cu at (32.8, 92.0)
- added R11: 10k, Resistor_SMD:R_0805_2012Metric, B.Cu at (32.8, 104.7)
- added R12: 10k, Resistor_SMD:R_0805_2012Metric, B.Cu at (32.8, 117.4)
- added R13: 10k, Resistor_SMD:R_0805_2012Metric, B.Cu at (126.0, 24.1)
- added R14: 10k, Resistor_SMD:R_0805_2012Metric, B.Cu at (113.3, 24.1)
- added R15: 10k, Resistor_SMD:R_0805_2012Metric, B.Cu at (100.6, 24.1)
- added R16: 10k, Resistor_SMD:R_0805_2012Metric, B.Cu at (193.9, 117.4)
- added R17: 10k, Resistor_SMD:R_0805_2012Metric, B.Cu at (193.9, 104.7)
- added R18: 10k, Resistor_SMD:R_0805_2012Metric, B.Cu at (193.9, 92.0)
- added R7: 10k, Resistor_SMD:R_0805_2012Metric, B.Cu at (100.6, 185.3)
- added R8: 10k, Resistor_SMD:R_0805_2012Metric, B.Cu at (113.3, 185.3)
- added R9: 10k, Resistor_SMD:R_0805_2012Metric, B.Cu at (126.0, 185.3)
- BZ1, R1: moved to B.Cu
- Q2: value BC847 -> MMBT2222A
- SW13: footprint Connector_PinHeader_2.54mm:PinHeader_1x02_P2.54mm_Vertical -> Library:Switch
- U3: value ~ -> PCF8575; moved to B.Cu
- moved U3 177.5 mm to (72.0, 63.5), turned to -45 degrees
- moved Q3 113.5 mm to (156.5, 63.0), turned to -45 degrees
- moved Q1 112.9 mm to (152.5, 66.5), turned to -45 degrees
- moved Q2 108.7 mm to (162.5, 57.0), turned to -45 degrees
- moved R6 104.3 mm to (149.0, 63.0), turned to 45 degrees
- moved R4 97.4 mm to (159.0, 53.5), turned to 45 degrees
- moved R2 97.1 mm to (153.0, 59.5), turned to 45 degrees
- moved R3 97.0 mm to (156.0, 56.5), turned to 45 degrees
- moved R5 95.4 mm to (159.4, 59.6), turned to -135 degrees
- moved BZ1 92.9 mm to (165.1, 145.0)
- moved SW13 86.1 mm to (138.0, 47.5)
- moved U2 46.9 mm to (175.1, 41.4), turned to -45 degrees
- moved R1 36.4 mm to (169.5, 70.5), turned to -90 degrees
Connections:
- U2 pad 12: unconnected-(U2-BAT-Pad12) -> +BATT
Routing:
- net /B8: track 0.00 -> 7.92 mm
- net /B9: track 0.00 -> 7.88 mm
- net /B7: track 0.00 -> 7.84 mm
Other:
- outline, holes or cut-outs redrawn
- board text added: "POWER"

Commit message: update
Parts:
- R1: moved to F.Cu
- moved R10 3.25 mm to (29.5, 92.0), turned to 0 degrees
- moved R11 3.25 mm to (29.5, 104.7), turned to 0 degrees
- moved R12 3.25 mm to (29.5, 117.4), turned to 0 degrees
- moved R13 3.23 mm to (126.0, 20.9), turned to -90 degrees
- moved R14 3.23 mm to (113.3, 20.9), turned to -90 degrees
- moved R15 3.23 mm to (100.6, 20.9), turned to -90 degrees
- moved R7 3.15 mm to (100.6, 188.5), turned to 90 degrees
- moved R8 3.15 mm to (113.3, 188.5), turned to 90 degrees
- moved R9 3.15 mm to (126.0, 188.5), turned to 90 degrees
- moved R16 3.13 mm to (197.0, 117.4), turned to 180 degrees
- moved R17 3.13 mm to (197.0, 104.7), turned to 180 degrees
- moved R18 3.13 mm to (197.0, 92.0), turned to 180 degrees
Routing:
- net +3.3V: track 0.00 -> 645.5 mm
- net VCC: track 0.00 -> 550.4 mm
- net /B10: track 0.00 -> 180.4 mm, vias 0 -> 2
- net Net-(D1-DIN): track 0.00 -> 176.4 mm
- net /B11: track 0.00 -> 172.5 mm, vias 0 -> 2
- net Net-(D5-DOUT): track 0.00 -> 168.2 mm
- net /B12: track 0.00 -> 165.8 mm, vias 0 -> 2
- net Net-(D10-DIN): track 0.00 -> 157.3 mm, vias 0 -> 2
- net Net-(BZ1--): track 0.00 -> 124.9 mm, vias 0 -> 2
- net /B6: track 0.00 -> 96.3 mm
- net /IRQ: track 0.00 -> 93.1 mm
- net /B5: track 0.00 -> 81.8 mm
- net /B7: track 7.84 -> 81.9 mm, vias 0 -> 1
- net /I2C2_SCL: track 0.00 -> 70.2 mm
- net /B4: track 0.00 -> 65.5 mm
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
Commit message: update
Parts:
- removed the D1 at (69.0, 155.8)
- moved BZ1 7.81 mm to (162.3, 152.3), turned to 135 degrees
- moved SW13 5.83 mm to (135.0, 52.5)
- moved U2 1.21 mm to (175.5, 42.5)
- renumbered D17 to D1, D8 to D10, D7 to D11, D6 to D12, D12 to D14, D11 to D15, D10 to D16, D16 to D2, D15 to D3, D14 to D4, D4 to D6, D3 to D7, D2 to D8, SW12 to SW1, SW9 to SW10, SW8 to SW11, SW7 to SW12, SW11 to SW2, SW10 to SW3, SW3 to SW4, SW2 to SW5, SW1 to SW6, SW6 to SW7, SW5 to SW8, SW4 to SW9
Connections:
- D1 pad 2: unconnected-(D17-DOUT-Pad2) -> Net-(D1-DOUT)
- D12 pad 4: Net-(D5-DOUT) -> Net-(D12-DIN)
- D13 pad 2: Net-(D13-DOUT) -> Net-(D12-DIN)
- D16 pad 4: Net-(D10-DIN) (its old number) -> unconnected-(D16-DIN-Pad4)
- D4 pad 4: Net-(D13-DOUT) -> Net-(D4-DIN)
- D5 pad 2: Net-(D5-DOUT) -> Net-(D4-DIN)
- D8 pad 4: Net-(D1-DOUT) -> Net-(D8-DIN)
- D9 pad 2: Net-(D10-DIN) (its old number) -> Net-(D8-DIN)
- R1 pad 2: Net-(D1-DIN) (its old number) -> Net-(D1-DOUT)
- R10 pad 2: /B4 -> /B5
- R11 pad 2: /B5 -> /B4
- R12 pad 2: /B6 -> /B3
- R13 pad 2: /B7 -> /B8
- R14 pad 2: /B8 -> /B7
- R15 pad 2: /B9 -> /B6
- R7 pad 2: /B1 -> /B2
- R8 pad 2: /B2 -> /B1
- R9 pad 2: /B3 -> /B9
- SW10 pad 2: /B9 -> /B6
- SW11 pad 2: /B8 -> /B7
- SW12 pad 2: /B7 -> /B8
- SW4 pad 2: /B3 -> /B9
- SW5 pad 2: /B2 -> /B1
- SW6 pad 2: /B1 -> /B2
- SW7 pad 2: /B6 -> /B3
- SW8 pad 2: /B5 -> /B4
- SW9 pad 2: /B4 -> /B5
- U3 pad 13: /B9 -> /B10
- U3 pad 14: /B10 -> /B11
- U3 pad 15: /B11 -> /B12
- U3 pad 16: /B12 -> /B2
- U3 pad 17: unconnected-(U3-P12-Pad17) -> /B1
- U3 pad 18: unconnected-(U3-P13-Pad18) -> /B9
- U3 pad 5: /B1 -> unconnected-(U3-P0-Pad5)
- U3 pad 6: /B2 -> unconnected-(U3-P1-Pad6)
Routing:
- net Net-(D1-DIN) (its old number): track 176.4 -> 0.00 mm
- net Net-(D5-DOUT): track 168.2 -> 0.00 mm
- net /B1: track 6.50 -> 170.5 mm, vias 0 -> 2
- net Net-(D10-DIN) (its old number): track 157.3 -> 0.00 mm, vias 2 -> 0
- net /B2: track 6.50 -> 161.8 mm, vias 0 -> 2
- net +3.3V: track 645.5 -> 500.2 mm
- net Net-(BZ1--): track 124.9 -> 0.00 mm, vias 2 -> 0
- net /B9: track 69.0 -> 175.2 mm, vias 1 -> 2
- net /B3: track 6.50 -> 90.0 mm
- net /I2C2_SCL: track 70.2 -> 0.00 mm
- net /I2C2_SDA: track 61.6 -> 0.00 mm
- net Net-(D12-DIN): track 0.00 -> 60.2 mm
- net Net-(D8-DIN): track 0.00 -> 59.0 mm
- net Net-(D4-DIN): track 0.00 -> 57.1 mm
- net /B6: track 96.3 -> 61.4 mm
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Other:
- outline, holes or cut-outs redrawn
- board text removed: "DUMMY"
- board text removed: "SW9"

Commit message: update
Routing:
- net Net-(BZ1--): track 0.00 -> 88.4 mm, vias 0 -> 2
- net +3.3V: track 500.2 -> 577.1 mm
- net /I2C2_SCL: track 0.00 -> 68.5 mm
- net /I2C2_SDA: track 0.00 -> 61.7 mm
- net /DC: track 31.0 -> 33.1 mm
- net /B5: track 72.7 -> 70.9 mm
- net /B3: track 90.0 -> 89.2 mm
- net /B2: track 161.8 -> 162.6 mm
- net /RST: track 33.7 -> 34.3 mm
- net /B4: track 80.3 -> 79.8 mm
- net GND: vias 2 -> 5
Other:
- board text removed: "J1"

Commit message: update
Parts:
- removed R4: 10k, Resistor_SMD:R_0805_2012Metric
- removed R5: 1k, Resistor_SMD:R_0805_2012Metric
- R3: value 1k -> 680R
- R6: value 100R -> 680R
- moved R1 17.5 mm to (165.5, 53.5), turned to 135 degrees
Connections:
- D1 pad 2: Net-(D1-DOUT) -> unconnected-(D1-DOUT-Pad2)
- D16 pad 4: unconnected-(D16-DIN-Pad4) -> Net-(D16-DIN)
- Q3 pad 1: Net-(Q3-G) -> Net-(Q2-C)
- R1 pad 2: Net-(D1-DOUT) -> Net-(D16-DIN)
- R3 pad 1: /EN -> /BASE
- U2 pad 19: unconnected-(U2-A5-Pad19) -> /BASE
Routing:
- net Net-(D16-DIN): track 0.00 -> 31.5 mm, vias 0 -> 2
- net /BASE: track 0.00 -> 19.3 mm, vias 0 -> 1
- net Net-(D1-DOUT): track 11.5 -> 0.00 mm
- net /EN: track 22.6 -> 14.2 mm, vias 1 -> 0
- net /NEOPIXEL: track 5.68 -> 11.1 mm, vias 0 -> 1
- net Net-(Q2-C): track 11.8 -> 15.0 mm
- net Net-(Q3-G): track 2.77 -> 0.00 mm

Commit message: V3
Other:
- board text added: "SW9"
